File: kicad/hammerhead_0.0.1/hammerhead_drive_motor_controller.kicad_sch (KiCad schematic)
At the start: 10 parts, among them U3 MAX14870ETC_T

Commit message: move thirdparty models to thirdparty dir
Parts:
- U3: footprint MAX14870ETC_T:SON50P300X300X80-13N -> MAX14870ETC_T:21-0664B_MXM
Changed lines of the file:
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@@
 			)
 		)
-		(property "Footprint" "MAX14870ETC_T:SON50P300X300X80-13N"
+		(property "Footprint" "MAX14870ETC_T:21-0664B_MXM"
 			(at 143.51 118.11 0)
 			(effects
